File: receiver_pcb/reciever_pcb.sch (EAGLE design)
At the start: 1 part, among them X1 43160-1203

Commit message: new reciever sch
Parts:
- removed X1: 43160-1203, con-molex:43160-1203
- added C1, C2: 4.7nF, rcl:C-EUC0805
- added C3: 22nF, rcl:C-EUC0805
- added C4: 1.8nF, rcl:C-EUC0805
- added C5: 10uF, rcl:C-EUC0805
- added C6: 2.2uF, rcl:C-EUC0805
- added C7: 10nF, rcl:C-EUC0805
- added D1, D2, D3: 40V 2A, diode:MBRA340T3
- added D4: 39V, diode:ZENER-DIODESMB
- added L1: 15uH, rcl:L-EUL1812
- added LED1: (no value), led:LEDCHIP-LED0805
- added R1: 3.01K, rcl:R-EU_R0805
- added R2, R4, R5: 10K, rcl:R-EU_R0805
- added R3: thermistor, rcl:R-EU_0207/2V
- added R6: 220, rcl:R-EU_R0805
- added T1: (no value), transistor:-PNP-SOT23-BCE
- added U$1: LT4120, custom parts:LT4120
- added X2: (no value), con-ptr500:AK500/2
- added X3: (no value), con-molex:KK-156-3
Connections:
- new net +4.1V: T1.E, U$1.BAT, U$1.BATSNS, X3-1.S
- new net GND: C5.2, C6.2, D2.A, D4.A, LED1.C, R1.2, R3.1, U$1.GND, X2-2.KL, X3-2.S
- new net N$1: C1.2, C2.1, C3.2, C4.1, D1.A, D2.C, X2-1.KL
- new net N$10: R4.1, U$1.!FAULT
- new net N$11: LED1.A, R6.1
- new net N$12: R6.2, T1.C, X3-3.S
- new net N$2: C2.2, C4.2, D3.A
- new net N$3: C6.1, R2.2, U$1.FREQ, U$1.INTVCC
- new net N$4: C7.1, U$1.BOOST
- new net N$5: C7.2, L1.1, U$1.SW
- new net N$6: L1.2, U$1.CHSNS
- new net N$7: R1.1, U$1.PROG
- new net N$8: R2.1, R3.2, U$1.NTC
- new net N$9: R5.1, T1.B, U$1.!CHARGE
- new net VCC: C1.1, C3.1, C5.1, D1.C, D3.C, D4.C, R4.2, R5.2, U$1.IN, U$1.RUN
Other:
- note added: "!Charge"
- note added: "Coil IN"
- note added: "Do we need it to charge at 400mA?"
- note added: "GND"
- note added: "How do we make the termistor easily reusable in case of battery replacement?"
- note added: "Vbatt"
- note added: "as close as possible to LIPO pin"
- note added: "low ESR"

Commit message: 1st reciever pcb
Parts:
- added TP1, TP2: TPTP19R, testpad:TPTP19R
- added X1: (no value), con-ptr500:AK500/2
Connections:
- net +4.1V: now also X1-2.KL
- net GND: now also X1-1.KL
- net N$10: now also TP1.TP
- net N$9: now also TP2.TP
Changed lines of the file:
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@@
 <part name="SUPPLY5" library="supply2" deviceset="+4.1V" device=""/>
 <part name="GND7" library="supply1" deviceset="GND" device=""/>
+<part name="TP1" library="testpad" deviceset="TP" device="TP19R"/>
+<part name="TP2" library="testpad" deviceset="TP" device="TP19R"/>
+<part name="X1" library="con-ptr500" deviceset="AK500/2" device=""/>
+<part name="GND8" library="supply1" deviceset="GND" device=""/>
 </parts>
 <sheets>
@@
 <instance part="SUPPLY5" gate="P" x="106.68" y="76.2"/>
 <instance part="GND7" gate="1" x="106.68" y="27.94"/>
+<instance part="TP1" gate="G$1" x="134.62" y="76.2"/>
+<instance part="TP2" gate="G$1" x="132.08" y="53.34" rot="R180"/>
+<instance part="X1" gate="-1" x="193.04" y="50.8" rot="R180"/>
+<instance part="X1" gate="-2" x="193.04" y="55.88" rot="R180"/>
+<instance part="GND8" gate="1" x="187.96" y="45.72"/>
 </instances>
 <busses>
@@
 <pinref part="LED1" gate="G$1" pin="C"/>
 <wire x1="106.68" y1="30.48" x2="106.68" y2="33.02" width="0.1524" layer="91"/>
+</segment>
+<segment>
+<pinref part="X1" gate="-1" pin="KL"/>
+<pinref part="GND8" gate="1" pin="GND"/>
+<wire x1="187.96" y1="48.26" x2="187.96" y2="50.8" width="0.1524" layer="91"/>
 </segment>
 </net>
@@
 <wire x1="180.34" y1="60.96" x2="180.34" y2="68.58" width="0.1524" layer="91"/>
 <junction x="180.34" y="68.58"/>
+<pinref part="X1" gate="-2" pin="KL"/>
+<wire x1="180.34" y1="60.96" x2="187.96" y2="60.96" width="0.1524" layer="91"/>
+<wire x1="187.96" y1="60.96" x2="187.96" y2="55.88" width="0.1524" layer="91"/>
+<junction x="180.34" y="60.96"/>
 </segment>
 <segment>
@@
 <pinref part="R5" gate="G$1" pin="1"/>
 <pinref part="U$1" gate="G$1" pin="!CHARGE"/>
-<wire x1="121.92" y1="60.96" x2="137.16" y2="60.96" width="0.1524" layer="91"/>
+<wire x1="121.92" y1="60.96" x2="132.08" y2="60.96" width="0.1524" layer="91"/>
 <pinref part="T1" gate="G$1" pin="B"/>
+<wire x1="132.08" y1="60.96" x2="137.16" y2="60.96" width="0.1524" layer="91"/>
 <wire x1="121.92" y1="60.96" x2="111.76" y2="60.96" width="0.1524" layer="91"/>
 <junction x="121.92" y="60.96"/>
+<pinref part="TP2" gate="G$1" pin="TP"/>
+<wire x1="132.08" y1="55.88" x2="132.08" y2="60.96" width="0.1524" layer="91"/>
+<junction x="132.08" y="60.96"/>
 </segment>
 </net>
@@
 <pinref part="R4" gate="G$1" pin="1"/>
 <pinref part="U$1" gate="G$1" pin="!FAULT"/>
-<wire x1="129.54" y1="66.04" x2="137.16" y2="66.04" width="0.1524" layer="91"/>
-</segment>
-</net>
+<wire x1="129.54" y1="66.04" x2="134.62" y2="66.04" width="0.1524" layer="91"/>
+<pinref part="TP1" gate="G$1" pin="TP"/>
+<wire x1="134.62" y1="66.04" x2="137.16" y2="66.04" width="0.1524" layer="91"/>
+<wire x1="134.62" y1="73.66" x2="134.62" y2="66.04" width="0.1524" layer="91"/>
+<junction x="134.62" y="66.04"/>
+</segment>
+</net>
