File: charger_pcb/charger_pcb.sch (EAGLE design)
At the start: 17 parts

Commit message: emitter 1st pcb
Other:
- note added: "Coil OUT"
Changed lines of the file:
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@@
 <sheet>
 <plain>
+<text x="101.6" y="43.18" size="1.778" layer="97">Coil OUT</text>
 </plain>
 <instances>
