File: hardware/bbbbbb/bbbbbb.kicad_pcb (KiCad board)
At the start: 2 copper layers, 135.6 x 87.4 mm, 63 parts, among them P1 gondola charge, P2 enable pull up, Q1 Q_NPN_BEC, Q2 Q_NPN_BEC, Q4 Q_NPN_BEC, Q5 Q_NPN_BEC, U2 LTV-827, U3 LTV-827, U4 LTV-827, U7 ms0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

Commit message: footprints mostly done
Parts:
- removed Q4, Q5: Q_NPN_BEC, Housings_SOT-23_SOT-143_TSOT-6:SOT-23
- removed U7: ms0, Pin_Headers:Pin_Header_Straight_1x02
- removed U8: ms1, Pin_Headers:Pin_Header_Straight_1x02
- added C3: C, Capacitors_SMD:C_1206, F.Cu at (251.2, 141.5)
- added C4: C, Capacitors_SMD:C_1206, F.Cu at (242.8, 137.5)
- added Q3: BS170, TO_SOT_Packages_SMD:SOT-223, F.Cu at (237.6, 152.0)
- added R29: R, Resistors_SMD:R_1206, F.Cu at (246.6, 119.0)
- added R30: R, Resistors_SMD:R_1206, F.Cu at (244.7, 131.4)
- added U1: xbee, fp:xbee, F.Cu at (214.0, 129.0)
- added U5: drv2250, fp:drv8825, F.Cu at (173.7, 132.1)
- added U6: drv2250, fp:drv8825, F.Cu at (173.9, 109.3)
- added U9: LM358, fp:soic8, F.Cu at (252.5, 137.2)
- moved R27 41.4 mm to (202.4, 100.3)
- moved P2 41.4 mm to (206.5, 100.1)
- moved R28 41.4 mm to (215.5, 99.9)
- moved C1 33.8 mm to (172.7, 138.3)
- moved R15 31.2 mm to (206.0, 120.7)
- moved R18 31.2 mm to (186.9, 134.7)
- moved R19 31.2 mm to (187.1, 128.1)
- moved R7 31.2 mm to (205.6, 114.4)
- moved U2 31.2 mm to (196.2, 113.3)
- moved U3 31.2 mm to (196.5, 136.1)
- moved R14 31.2 mm to (205.7, 125.9)
- moved R16 31.2 mm to (186.8, 117.1)
- moved R17 31.2 mm to (186.9, 139.8)
- moved R20 31.2 mm to (187.1, 123.2)
- moved R8 31.2 mm to (206.0, 137.4)
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Connections:
- D6 pad 2: Net-(D6-Pad2) -> x-home
- D7 pad 2: Net-(D7-Pad2) -> y-home
- P1 pad 2: (no net) -> Net-(P1-Pad2)
- R12 pad 1: x-home -> Net-(C3-Pad2)
- R13 pad 1: y-home -> Net-(C4-Pad2)
- R23 pad 1: Net-(Q4-Pad1) -> +3V3
- R23 pad 2: x-home -> Net-(R23-Pad2)
- R24 pad 1: Net-(Q5-Pad1) -> Net-(R23-Pad2)
- R24 pad 2: y-home -> Earth
- R25 pad 2: Net-(D6-Pad2) -> Net-(R25-Pad2)
- R26 pad 1: +3V3 -> Net-(R25-Pad2)
- R26 pad 2: Net-(D7-Pad2) -> Earth
- ms0 pad 2: (no net) -> /ms0
- ms1 pad 2: (no net) -> /ms1
- port9 pad 24: (no net) -> /xbee-rx
- port9 pad 26: (no net) -> /xbee-tx
- port9 pad 44: Earth -> Net-(port9-Pad44)
- port9 pad 46: Earth -> Net-(port9-Pad44)
- step-x1 pad 1: (no net) -> Net-(U5-Pad14)
- step-x1 pad 2: (no net) -> Net-(U5-Pad13)
- step-x1 pad 3: (no net) -> Net-(U5-Pad12)
- step-x1 pad 4: (no net) -> Net-(U5-Pad11)
- step-y1 pad 1: (no net) -> Net-(U6-Pad14)
- step-y1 pad 2: (no net) -> Net-(U6-Pad13)
- step-y1 pad 3: (no net) -> Net-(U6-Pad12)
- step-y1 pad 4: (no net) -> Net-(U6-Pad11)
- x-home1 pad 3: x-home -> Net-(C3-Pad2)
- y-home1 pad 3: y-home -> Net-(C4-Pad2)

Commit message: gondola charge
Parts:
- removed Q2: Q_NPN_BEC, Housings_SOT-23_SOT-143_TSOT-6:SOT-23
- removed R4: R, Resistors_SMD:R_1206
- moved U9 97.7 mm to (163.0, 98.0)
- moved R26 95.5 mm to (163.0, 90.0), turned to 270 degrees
- moved R25 94.8 mm to (160.0, 90.0), turned to 90 degrees
- moved R23 91.7 mm to (161.0, 106.0), turned to 90 degrees
- moved C3 91.4 mm to (167.0, 106.0), turned to 90 degrees
- moved R24 90.8 mm to (164.0, 106.0), turned to 270 degrees
- moved C4 90.3 mm to (166.0, 90.0), turned to 90 degrees
- moved fan1 64.4 mm to (234.0, 154.0)
- moved R12 61.5 mm to (155.0, 88.0), turned to 0 degrees
- moved R10 55.7 mm to (154.0, 94.0), turned to 270 degrees
- moved D4 53.7 mm to (235.0, 148.0)
- moved x-home1 53.0 mm to (149.0, 95.0), turned to 180 degrees
- moved R1 47.2 mm to (235.0, 144.0)
- moved D7 34.6 mm to (217.0, 107.0)
- moved R30 33.5 mm to (223.0, 106.0)
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Connections:
- P1 pad 1: +24V -> +5V
- P1 pad 2: Net-(P1-Pad2) -> Net-(D4-Pad1)
- Q1 pad 2: Earth -> (no net)
- Q3 pad 1: Net-(P1-Pad2) -> Net-(D4-Pad1)
- R1 pad 1: Net-(Q2-Pad1) -> +5V
- R1 pad 2: gondola-charge -> Net-(D4-Pad2)
Other:
- board size 135.6 x 87.4 mm -> 123 x 74 mm

Commit message: silkscreen & values
Parts:
- removed P1: gondola charge, Connect:AK300-2
- removed P2: enable pull up, Pin_Headers:Pin_Header_Straight_1x03
- removed Q3: BS170, TO_SOT_Packages_SMD:SOT-223
- removed fan1: CONN_01X02, Pin_Headers:Pin_Header_Straight_1x02
- added 12v1: fan, Pin_Headers:Pin_Header_Straight_1x02, F.Cu at (234.0, 154.0)
- added C5: 47u, Capacitors_Elko_ThroughHole:Elko_vert_11.2x7.5mm_RM2.5, F.Cu at (220.0, 139.0)
- added P4: CONN_01X08, Pin_Headers:Pin_Header_Straight_1x08, F.Cu at (252.0, 112.0)
- added Q2: pmt29en, TO_SOT_Packages_SMD:SOT-223, F.Cu at (247.0, 142.0)
- added bb-5v1: bb-5v, Pin_Headers:Pin_Header_Straight_1x02, F.Cu at (251.0, 92.0)
- added en1: enable pull up, Pin_Headers:Pin_Header_Straight_1x03, F.Cu at (194.5, 99.0)
- added gondola1: gondola charge, Connect:AK300-2, F.Cu at (220.0, 151.0)
- added step-x2: CONN_01X04, Pin_Headers:Pin_Header_Straight_1x04, F.Cu at (150.0, 149.0)
- added step-y2: CONN_01X04, Pin_Headers:Pin_Header_Straight_1x04, F.Cu at (150.0, 125.0)
- 12/5v1: value CONN_01X03 -> 12/5v
- 7seg1: value CONN_01X08 -> 7seg
- C1, C2: value CP -> 47uf
- C3, C4: value C -> 2.2n
- Q1: value Q_NPN_BEC -> BC849C
- R1, R5: value R -> 560
- R10, R11: value R -> 330
- R12, R13, R6: value R -> 1k
- R2: value R -> 4.7k
- R21, R29, R30: value R -> 220
- R22, R27, R28: value R -> 10k
- R23, R25: value R -> 8k
- R24, R26, R3: value R -> 2k
- buttons1: value CONN_01X04 -> buttons
- servo1: value CONN_01X03 -> servo
- moved D7 17.8 mm to (231.0, 96.0)
- moved D6 13.5 mm to (239.0, 96.0)
- moved R30 8.94 mm to (231.0, 102.0)
- moved R29 6.08 mm to (239.0, 102.0)
- moved U1 5.10 mm to (219.0, 123.0)
- moved R1 3.61 mm to (233.0, 141.0)
- moved R22 3.61 mm to (239.0, 142.0), turned to 270 degrees
- moved 24v1 3.00 mm to (188.0, 151.0)
- moved D4 2.83 mm to (233.0, 146.0)
- moved R6 1.76 mm to (223.0, 101.0)
Connections:
- Q1 pad 2: (no net) -> Earth
- port9 pad 23: (no net) -> /gpio1
- port9 pad 25: (no net) -> /gpio2
- port9 pad 27: (no net) -> /gpio3
- port9 pad 29: (no net) -> /gpio4
- port9 pad 31: (no net) -> /gpio5
- port9 pad 5: (no net) -> /bb-5v
- port9 pad 6: (no net) -> /bb-5v
Routing:
- net Earth: track 0.00 -> 605.8 mm, vias 0 -> 9
- net +3V3: track 0.00 -> 291.0 mm, vias 0 -> 8
- net +5V: track 0.00 -> 229.9 mm, vias 0 -> 4
- net +12V: track 0.00 -> 145.4 mm
- net x-home: track 0.00 -> 142.9 mm, vias 0 -> 6
- net /7seg-clk: track 0.00 -> 138.3 mm
- net /7seg-!oe: track 0.00 -> 135.4 mm, vias 0 -> 3
- net +24V: track 0.00 -> 131.8 mm
- net enable: track 0.00 -> 130.9 mm, vias 0 -> 2
- net y-home: track 0.00 -> 129.3 mm, vias 0 -> 5
- net /7seg-sdo: track 0.00 -> 123.6 mm, vias 0 -> 2
- net /enable-ext: track 0.00 -> 120.2 mm, vias 0 -> 1
- net /7seg-le: track 0.00 -> 111.4 mm
- net /xstep-ext: track 0.00 -> 84.8 mm
- net /xdir-ext: track 0.00 -> 77.6 mm, vias 0 -> 2
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- added copper zone on B.Cu, net Earth
- added copper zone on F.Cu, net Earth
Other:
- net class power added: clearance 0.2, trace_width 1, via_dia 0.6, via_drill 0.4
- board text added: "3.3v, p1, p2, p3, p4, p5, 0v, 0v"
- board text added: "bbbbbb v0.1 6/2016"
