File: hardware/bbbbbb_pcb/bbbbbb.kicad_pcb (KiCad board)
At the start: 2 copper layers, 123 x 74 mm, 71 parts, among them P4 CONN_01X08, Q1 BC849C, Q2 pmt29en, U1 xbee, U2 LTV-827, U3 LTV-827, U4 LTV-827, U5 drv2250, U6 drv2250, U9 LM358

Commit message: oshpark fab
Parts:
- added 12v sol 5v: sol sel, Pin_Headers:Pin_Header_Straight_1x03, F.Cu at (240.8, 149.0)
- added C6: C, Capacitors_SMD:C_1206, F.Cu at (233.2, 135.0)
- added R31: R, Resistors_SMD:R_1206, F.Cu at (234.0, 119.0)
- added R32: R, Resistors_SMD:R_1206, F.Cu at (233.0, 131.5)
- added REF**: MountingHole_3mm, Mounting_Holes:MountingHole_3mm, F.Cu at (187.0, 95.5)
- added REF**: MountingHole_3mm, Mounting_Holes:MountingHole_3mm, F.Cu at (248.2, 134.2)
- added REF**: MountingHole_3mm, Mounting_Holes:MountingHole_3mm, F.Cu at (245.5, 92.0)
- added REF**: MountingHole_3mm, Mounting_Holes:MountingHole_3mm, F.Cu at (173.2, 139.5)
- added U7: tcn75, Housings_SSOP:MSOP-8_3x3mm_Pitch0.65mm, F.Cu at (233.8, 125.2)
- added pwm1: CONN_01X01, Pin_Headers:Pin_Header_Straight_1x01, F.Cu at (181.0, 92.2)
- added solenoids: solenoids, Pin_Headers:Pin_Header_Straight_1x02, F.Cu at (241.5, 154.0)
- 0v 12v 5v: renamed from 12/5v1
- 0v 24v: renamed from 24v1
- bbb 5v: renamed from bb-5v1
- moved D2 13.4 mm to (256.5, 149.2)
- moved R3 13.2 mm to (256.5, 153.8)
- moved D1 4.37 mm to (262.8, 149.5)
- moved R2 4.21 mm to (262.5, 153.8)
- moved R5 1.25 mm to (250.5, 153.5)
- moved D3 0.75 mm to (250.5, 149.2)
- moved D5 0.50 mm to (217.5, 96.0)
- renumbered buttons1 to buttons, gondola1 to gondola, servo1 to servo, step-x1 to step-x, step-y1 to step-y, x-ext1 to x-ext, x-home1 to x-home, y-ext1 to y-ext, y-home1 to y-home
Connections:
- port9 pad 19: (no net) -> scl
- port9 pad 20: (no net) -> sda
Routing:
- net Earth: track 605.8 -> 683.6 mm, vias 9 -> 15
- net +3V3: track 291.0 -> 336.8 mm, vias 8 -> 11
- net sda: track 0.00 -> 45.6 mm, vias 0 -> 1
- net scl: track 0.00 -> 45.3 mm, vias 0 -> 3
- net +12V: track 145.4 -> 163.2 mm
- net +5V: track 229.9 -> 246.2 mm, vias 4 -> 3
- net /7seg-!oe: track 135.4 -> 150.6 mm
- net +24V: track 131.8 -> 139.4 mm
- net Net-(sol1-Pad2): track 0.00 -> 5.74 mm
- net /butt-power: track 22.8 -> 28.4 mm
- net /butt-estop: track 26.5 -> 30.1 mm
- net /butt-reset: track 32.0 -> 34.4 mm
- net y-home: track 129.3 -> 130.6 mm
- net Net-(D3-Pad2): track 4.84 -> 4.26 mm
Other:
- outline, holes or cut-outs redrawn
- board text added: "5v 12v 24v"
- board text added: "bbbbbb v2 6/2016"
- board text added: "bbbbbb v2 matt venn 2016"
- board text added: "enable"
- board text added: "fan"
- board text added: "home y x"
- board text added: "led pwm"
- board text added: "made with love in Spain!"
- board text removed: "bbbbbb v0.1 6/2016"
